File: hardware/BREAD_Slice.kicad_pcb (KiCad board)
At the start: 4 copper layers, 100.1 x 144.9 mm, 16 parts, among them J1 Conn_01x10_Female, U1 AP63205, U2 NUCLEO-L432KC

Commit message: review and revise board and update footprints
Parts:
- D1: footprint SparkFun-LED:WS2812-5050-4PIN -> KMLib_IC_SMD:WS2812-5050-4PIN
- HS1: footprint kml-custom:Thermal Pad -> KMLib_Mounting:Thermal Pad
- U2: footprint kml-custom:MODULE_NUCLEO-L432KC -> KMLib_Boards_Modules:MODULE_NUCLEO-L432KC
Routing:
- net +12V: track 48.2 -> 51.2 mm, vias 0 -> 1
- net /I2C_DAT: track 44.9 -> 47.5 mm
- net /I2C_CLK: track 45.5 -> 46.5 mm
