File: hardware/BREAD_Slice.kicad_sch (KiCad schematic)
At the start: 15 parts, among them J1 Conn_01x10_Female, U1 AP63205

Commit message: initial commit post-fork from s2l
Parts:
- removed A1: Arduino_Nano_v3.x, Module:Arduino_Nano, symbol MCU_Module:Arduino_Nano_v3.x
- added U2: NUCLEO-L432KC, kml-custom:MODULE_NUCLEO-L432KC, symbol kml-custom:NUCLEO-L432KC
Connections:
- net ESTOP: now also U2.CN3_5 (PA12)
- net I2C_CLK: now also U2.CN4_7 (PA6)
- net I2C_DAT: now also U2.CN4_8 (PA5)
- net INT: now also U2.CN3_6 (PB0)
- net LED: now also U2.CN3_8 (PB6)
- net SYNC: now also U2.CN3_7 (PB7)
- net +5V renamed +5VD
- net +5VD: now also U2.CN4_4 (+5V)
- net GND renamed GNDD
- net GNDD: now also U2.CN3_4 (GND_CN3), U2.CN4_2 (GND_CN4)
- new net +3V3: U2.CN4_14 (+3V3)
- no-connect marks 22 -> 24
Other:
- note added: "Digital 5V"
- note added: "ON OFF ON ON ON ON OFF OFF"
- note added: "Pinout Details: STM32 Nucleo-32 L432KC ------------------------------------------------------------------------------------- Pin | Function | Notes ------------------------------------------------------------------------------------- VIN | External Supply Input | 7-12V input via CN4 pin 1; powers onboard 3.3V regulator GND | Ground | Ground reference (multiple available) NRST | Reset Input | Acti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"
- note added: "SB10 (VREF+) - ON: VREF+ on STM32 is connected to VDD. - OFF: VREF+ on STM32 is not connected to VDD and it is provided by pin 13 of CN4. SB15 (LD3-LED) - ON: Green user LED LD3 is connected to D13 of ARDUINO® Nano signal. - OFF: Green user LED LD3 is not connected. SB9 (NRST) - ON: The NRST signal of ST-LINK is connected to the NRST pin of the STM32. - OFF: The NRST signal of ST-LINK is not conn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"
- note added: "STM32 NUCLEO32 STM32L432KC"
- note added: "internal note: removed int to move estop to make room on D2"
- note removed: "5V Switching Supply"
- note removed: "Arduino Nano"
- note removed: "Pinout Details Arduino Nano: -------------------------------------------------------------------------------------------------------------------- Pin | Function | Limitations/Notes -------------------------------------------------------------------------------------------------------------------- VIN | External Supply Input | External power source 7-12V GND | Ground | First GND pin available for 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"
- moved on the sheet: C1, C2, C3, C4, D1, H1, H2, H3, H4, J1, L1, U1
