File: hardware/BREAD_Slice.kicad_sch (KiCad schematic)
At the start: 15 parts, among them J1 Conn_01x10_Female, U1 AP63205, U2 NUCLEO-L432KC

Commit message: review and revise board and update footprints
Parts:
- D1: footprint SparkFun-LED:WS2812-5050-4PIN -> KMLib_IC_SMD:WS2812-5050-4PIN
- HS1: footprint kml-custom:Thermal Pad -> KMLib_Mounting:Thermal Pad
- U2: footprint kml-custom:MODULE_NUCLEO-L432KC -> KMLib_Boards_Modules:MODULE_NUCLEO-L432KC
Changed lines of the file:
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@@
 			)
 		)
-		(property "Footprint" "kml-custom:Thermal Pad"
+		(property "Footprint" "KMLib_Mounting:Thermal Pad"
 			(at 34.5948 95.25 0)
 			(effects
@@
 			)
 		)
-		(property "Footprint" "kml-custom:MODULE_NUCLEO-L432KC"
+		(property "Footprint" "KMLib_Boards_Modules:MODULE_NUCLEO-L432KC"
 			(at 39.37 137.16 0)
 			(effects
@@
 			)
 		)
-		(property "Footprint" "SparkFun-LED:WS2812-5050-4PIN"
+		(property "Footprint" "KMLib_IC_SMD:WS2812-5050-4PIN"
 			(at 12.7 40.64 0)
 			(effects
@@
 			)
 		)
-		(property "Footprint" "kml-custom:MODULE_NUCLEO-L432KC"
+		(property "Footprint" "KMLib_Boards_Modules:MODULE_NUCLEO-L432KC"
 			(at 39.37 173.99 0)
 			(effects
